File: arduStep.kicad_sch (KiCad schematic)
At the start: 3 parts

Commit message: edit cajetin
Parts:
- added C1: 10nf, Capacitor_SMD:C_1206_3216Metric, symbol Device:C_Polarized
- added J2: jst battery, Connector_JST:JST_XH_S2B-XH-A_1x02_P2.50mm_Horizontal, symbol Connector:Conn_01x02_Male
- J1: renamed from J?; value jst 4pin -> stepper; footprint (none) -> Connector_JST:JST_XH_S4B-XH-A_1x04_P2.50mm_Horizontal
- U1: renamed from U?; footprint (none) -> Package_DIP:DIP-16_W7.62mm
- gave numbers to parts that had none: 1
Connections:
- net GND: now also C1.2, J2.2 (Pin_2)
- net in1: now also A1.7 (D4); no longer A1.5 (D2)
- net in2: now also A1.8 (D5); no longer A1.6 (D3)
- net in3: now also A1.9 (D6); no longer A1.7 (D4)
- net in4: now also A1.10 (D7); no longer A1.8 (D5)
- net 5V: now reaches U1.9 (COM)
- net 5V: now also C1.1, J2.1 (Pin_1)
Other:
- moved on the sheet: J1, U1
